Commit message: Prepare conference paper repository release

File: src/ur5e_sim/urdf/camera.xacro (robot description, xacro)
@@ -15,5 +15,5 @@
             <geometry>
                 <!-- <box size="0.01 0.03 0.03" /> -->
-                <mesh filename="package://ur5e_sim/meshes/sensors/camera/kinetic.stl"/>
+                <mesh filename="file://${URYT}/meshes/sensors/camera/kinetic.stl"/>
             </geometry>
             <material name="red"/>
@@ -21,5 +21,5 @@
         <collision>
             <geometry>
-                <mesh filename="package://ur5e_sim/meshes/sensors/camera/kinetic.dae"/>
+                <mesh filename="file://${URYT}/meshes/sensors/camera/kinetic.dae"/>
             </geometry>
         </collision>
@@ -29,5 +29,5 @@
         <parent link="base_link"/>
         <child link="camera_link"/>
-        <origin xyz="0.5 0 1.2" rpy="0 1.57 0" />
+        <origin xyz="0.305 0.350 0.952" rpy="0 1.57 0" />
     </joint>
     <link name="camera_optical_link"></link>

File: src/ur5e_sim/urdf/robotiq_gripper_macro.xacro (robot description, xacro)
@@ -43,10 +43,10 @@
             <visual>
                 <geometry>
-                    <mesh filename="package://robotiq_description/meshes/visual/2f_85/robotiq_base.dae" />
-                </geometry>
-            </visual>
-            <collision>
-                <geometry>
-                    <mesh filename="package://robotiq_description/meshes/collision/2f_85/robotiq_base.stl" />
+                    <mesh filename="file://${ROBI}/meshes/visual/2f_85/robotiq_base.dae"/>
+                </geometry>
+            </visual>
+            <collision>
+                <geometry>
+                    <mesh filename="file://${ROBI}/meshes/collision/2f_85/robotiq_base.stl"/>
                 </geometry>
             </collision>
@@ -60,10 +60,10 @@
             <visual>
                 <geometry>
-                    <mesh filename="package://robotiq_description/meshes/visual/2f_85/left_knuckle.dae" />
-                </geometry>
-            </visual>
-            <collision>
-                <geometry>
-                    <mesh filename="package://robotiq_description/meshes/collision/2f_85/left_knuckle.stl" />
+                    <mesh filename="file://${ROBI}/meshes/visual/2f_85/left_knuckle.dae" />
+                </geometry>
+            </visual>
+            <collision>
+                <geometry>
+                    <mesh filename="file://${ROBI}/meshes/collision/2f_85/left_knuckle.stl" />
                 </geometry>
             </collision>
@@ -77,10 +77,10 @@
             <visual>
                 <geometry>
-                    <mesh filename="package://robotiq_description/meshes/visual/2f_85/right_knuckle.dae" />
-                </geometry>
-            </visual>
-            <collision>
-                <geometry>
-                    <mesh filename="package://robotiq_description/meshes/collision/2f_85/right_knuckle.stl" />
+                    <mesh filename="file://${ROBI}/meshes/visual/2f_85/right_knuckle.dae" />
+                </geometry>
+            </visual>
+            <collision>
+                <geometry>
+                    <mesh filename="file://${ROBI}/meshes/collision/2f_85/right_knuckle.stl" />
                 </geometry>
             </collision>
@@ -94,10 +94,10 @@
             <visual>
                 <geometry>
-                    <mesh filename="package://robotiq_description/meshes/visual/2f_85/left_finger.dae" />
-                </geometry>
-            </visual>
-            <collision>
-                <geometry>
-                    <mesh filename="package://robotiq_description/meshes/collision/2f_85/left_finger.stl" />
+                    <mesh filename="file://${ROBI}/meshes/visual/2f_85/left_finger.dae" />
+                </geometry>
+            </visual>
+            <collision>
+                <geometry>
+                    <mesh filename="file://${ROBI}/meshes/collision/2f_85/left_finger.stl" />
                 </geometry>
             </collision>
@@ -111,10 +111,10 @@
             <visual>
                 <geometry>
-                    <mesh filename="package://robotiq_description/meshes/visual/2f_85/right_finger.dae" />
-                </geometry>
-            </visual>
-            <collision>
-                <geometry>
-                    <mesh filename="package://robotiq_description/meshes/collision/2f_85/right_finger.stl" />
+                    <mesh filename="file://${ROBI}/meshes/visual/2f_85/right_finger.dae" />
+                </geometry>
+            </visual>
+            <collision>
+                <geometry>
+                    <mesh filename="file://${ROBI}/meshes/collision/2f_85/right_finger.stl" />
                 </geometry>
             </collision>
@@ -128,10 +128,10 @@
             <visual>
                 <geometry>
-                    <mesh filename="package://robotiq_description/meshes/visual/2f_85/left_inner_knuckle.dae" />
-                </geometry>
-            </visual>
-            <collision>
-                <geometry>
-                    <mesh filename="package://robotiq_description/meshes/collision/2f_85/left_inner_knuckle.stl" />
+                    <mesh filename="file://${ROBI}/meshes/visual/2f_85/left_inner_knuckle.dae" />
+                </geometry>
+            </visual>
+            <collision>
+                <geometry>
+                    <mesh filename="file://${ROBI}/meshes/collision/2f_85/left_inner_knuckle.stl" />
                 </geometry>
             </collision>
@@ -145,10 +145,10 @@
             <visual>
                 <geometry>
-                    <mesh filename="package://robotiq_description/meshes/visual/2f_85/right_inner_knuckle.dae" />
-                </geometry>
-            </visual>
-            <collision>
-                <geometry>
-                    <mesh filename="package://robotiq_description/meshes/collision/2f_85/right_inner_knuckle.stl" />
+                    <mesh filename="file://${ROBI}/meshes/visual/2f_85/right_inner_knuckle.dae" />
+                </geometry>
+            </visual>
+            <collision>
+                <geometry>
+                    <mesh filename="file://${ROBI}/meshes/collision/2f_85/right_inner_knuckle.stl" />
                 </geometry>
             </collision>
@@ -162,10 +162,10 @@
             <visual>
                 <geometry>
-                    <mesh filename="package://robotiq_description/meshes/visual/2f_85/left_finger_tip.dae" />
-                </geometry>
-            </visual>
-            <collision>
-                <geometry>
-                    <mesh filename="package://robotiq_description/meshes/collision/2f_85/left_finger_tip.stl" />
+                    <mesh filename="file://${ROBI}/meshes/visual/2f_85/left_finger_tip.dae" />
+                </geometry>
+            </visual>
+            <collision>
+                <geometry>
+                    <mesh filename="file://${ROBI}/meshes/collision/2f_85/left_finger_tip.stl" />
                 </geometry>
                 <surface>
@@ -197,10 +197,10 @@
             <visual>
                 <geometry>
-                    <mesh filename="package://robotiq_description/meshes/visual/2f_85/right_finger_tip.dae" />
-                </geometry>
-            </visual>
-            <collision>
-                <geometry>
-                    <mesh filename="package://robotiq_description/meshes/collision/2f_85/right_finger_tip.stl" />
+                    <mesh filename="file://${ROBI}/meshes/visual/2f_85/right_finger_tip.dae" />
+                </geometry>
+            </visual>
+            <collision>
+                <geometry>
+                    <mesh filename="file://${ROBI}/meshes/collision/2f_85/right_finger_tip.stl" />
                 </geometry>
                 <surface>

File: src/ur5e_sim/urdf/ur5_camera_gripper.urdf.xacro (robot description, xacro)
@@ -4,4 +4,6 @@
    <xacro:arg name="name" default="ur"/>
    <!-- import main macro -->
+   <xacro:property name="URYT" value="$(find ur5e_sim)"/>
+   <xacro:property name="ROBI" value="$(find robotiq_description)"/>
    <xacro:include filename="$(find ur5e_sim)/urdf/camera.xacro"/>
    <xacro:include filename="$(find ur5e_sim)/urdf/ur5_macro.xacro"/>
@@ -116,5 +118,5 @@
      trajectory_port="$(arg trajectory_port)"
      >
-     <origin xyz="0 0 0.8" rpy="0 0 0" />          <!-- position robot in the world -->
+     <origin xyz="0 0 0.73" rpy="0 0 0" />          <!-- position robot in the world -->
    </xacro:ur_robot>
    <xacro:if value="$(arg sim_gazebo)">
